File: Hardware/Mutatio/Mutatio_REV1.brd (EAGLE design)
At the start: 47.2 x 50 mm, 45 parts, among them IC1 OPA743, IC2 74AUC1G14DBV, IC3 MCP1703CB, J1 MICRO-SDCARD-CONNECTOR-330006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

Commit message: Added bug description and changed component values
Parts:
- C5: value NC -> 1uF
- D4, D5: value (none) -> NC
- R1: value 100k -> 51k
- R2: value 100k -> 100k||51k
- R3: value 10k -> 1k
- R7: value 10k -> 0R
Changed lines of the file:
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@@
 <setting verticaltext="up"/>
 </settings>
-<grid distance="10" unitdist="mm" unit="mm" style="lines" multiple="1" display="yes" altdistance="0.1" altunitdist="mm" altunit="mm"/>
+<grid distance="393.700787" unitdist="mil" unit="mil" style="lines" multiple="1" display="yes" altdistance="0.1" altunitdist="mm" altunit="mm"/>
 <layers>
 <layer number="1" name="Top" color="4" fill="1" visible="yes" active="yes"/>
@@
 <attribute name="VALUE" x="8.232" y="16.711" size="1.27" layer="27" rot="R90"/>
 </element>
-<element name="R1" library="resistor" package="R0603" value="100k" x="10.6" y="17.6" smashed="yes" rot="R270">
+<element name="R1" library="resistor" package="R0603" value="51k" x="10.6" y="17.6" smashed="yes" rot="R270">
 <attribute name="NAME" x="10.111" y="19.289" size="0.8128" layer="25" font="vector" ratio="20"/>
 <attribute name="VALUE" x="8.568" y="18.489" size="1.27" layer="27" rot="R270"/>
 </element>
-<element name="R2" library="resistor" package="R0603" value="100k" x="8.4" y="17.6" smashed="yes" rot="R90">
+<element name="R2" library="resistor" package="R0603" value="100k||51k" x="8.4" y="17.6" smashed="yes" rot="R90">
 <attribute name="NAME" x="9.289" y="19.911" size="0.8128" layer="25" font="vector" ratio="20" rot="R180"/>
 <attribute name="VALUE" x="10.432" y="16.711" size="1.27" layer="27" rot="R90"/>
@@
 <attribute name="VALUE" x="11.413" y="11.149" size="1.27" layer="27" rot="R90"/>
 </element>
-<element name="R3" library="resistor" package="R0603" value="10k" x="3.6" y="8.8" smashed="yes" rot="R270">
+<element name="R3" library="resistor" package="R0603" value="1k" x="3.6" y="8.8" smashed="yes" rot="R270">
 <attribute name="NAME" x="2.911" y="10.489" size="0.8128" layer="25" font="vector" ratio="20"/>
 <attribute name="VALUE" x="1.568" y="9.689" size="1.27" layer="27" rot="R270"/>
@@
 <attribute name="VALUE" x="-0.432" y="6.489" size="1.27" layer="27" rot="R270"/>
 </element>
-<element name="R7" library="resistor" package="R0603" value="10k" x="3.6" y="5.6" smashed="yes" rot="R270">
+<element name="R7" library="resistor" package="R0603" value="0R" x="3.6" y="5.6" smashed="yes" rot="R270">
 <attribute name="NAME" x="4.289" y="5.889" size="0.8128" layer="25" font="vector" ratio="20" rot="R270"/>
 <attribute name="VALUE" x="1.568" y="6.489" size="1.27" layer="27" rot="R270"/>
@@
 <attribute name="VALUE" x="-0.432" y="3.289" size="1.27" layer="27" rot="R270"/>
 </element>
-<element name="C5" library="resistor" package="C0603" value="NC" x="1.6" y="8.8" smashed="yes" rot="R270">
+<element name="C5" library="resistor" package="C0603" value="1uF" x="1.6" y="8.8" smashed="yes" rot="R270">
 <attribute name="NAME" x="0.911" y="10.562" size="0.8128" layer="25" font="vector" ratio="20"/>
 <attribute name="VALUE" x="-0.432" y="9.689" size="1.27" layer="27" rot="R270"/>
@@
 <attribute name="VALUE" x="13.813" y="5.149" size="1.27" layer="27" rot="R90"/>
 </element>
-<element name="D4" library="diode" package="MINIMELF" value="" x="9" y="6.8" smashed="yes" rot="R90">
+<element name="D4" library="diode" package="MINIMELF" value="NC" x="9" y="6.8" smashed="yes" rot="R90">
 <attribute name="NAME" x="9.851" y="4.057" size="0.8128" layer="25" font="vector" ratio="20" rot="R180"/>
 <attribute name="VALUE" x="11.413" y="5.149" size="1.27" layer="27" rot="R90"/>
 </element>
-<element name="D5" library="diode" package="MINIMELF" value="" x="6.4" y="12.8" smashed="yes" rot="R90">
+<element name="D5" library="diode" package="MINIMELF" value="NC" x="6.4" y="12.8" smashed="yes" rot="R90">
 <attribute name="NAME" x="7.251" y="16.087" size="0.8128" layer="25" font="vector" ratio="20" rot="R180"/>
 <attribute name="VALUE" x="8.813" y="11.149" size="1.27" layer="27" rot="R90"/>

Commit message: Added bug description and changed component values
Parts:
- C9: value 1uF -> 22uF
Changed lines of the file:
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@@
 </element>
 <element name="U$1" library="DS3231_Module" package="DS3231_MODULE_BIGCON" value="DS3231_MODULEBIG_CONNECTER_ONLY" x="22.8" y="20.4" smashed="yes" rot="MR90"/>
-<element name="C9" library="resistor" package="C0603" value="1uF" x="6.2" y="17.6" smashed="yes" rot="R90">
+<element name="C9" library="resistor" package="C0603" value="22uF" x="6.2" y="17.6" smashed="yes" rot="R90">
 <attribute name="NAME" x="7.089" y="20.038" size="0.8128" layer="25" font="vector" ratio="20" rot="R180"/>
 <attribute name="VALUE" x="8.232" y="16.711" size="1.27" layer="27" rot="R90"/>
