File: Hardware/Mutatio/Mutatio_REV2.sch (EAGLE design)
At the start: 35 parts, among them IC1 DS3231/SO, IC2 74AUC1G14DBV, J1 MICRO-SDCARD-CONNECTOR-330006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

Commit message: finished revision 2
Parts:
- removed C11: 100uF, resistor:C-EUC1206
- added D6: (no value), diode:DIODE-MINIMELF
Connections:
- new net N$6: C10.1, D6.C, IC1.VBAT
- net +3V3: no longer C10.1, C11.1, IC1.VBAT
- net +5V: now also D6.A
- net GND: no longer C11.2
Other:
- note added: "RTC Option 1:"
- note added: "RTC Option 2:"
- moved on the sheet: C1, C10, C2, C3, C4, C6, C7, C8, IC1, J1, LED, R4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

Commit message: Updated REV2 hardware
changed the Signal and the LED pin so upload and bootup works properly
Connections:
- net SIGNAL: now also U$2.D8; no longer U$2.D4
- net WS2812_DATA: now also U$2.D4; no longer U$2.D8
Changed lines of the file:
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@@
 <net name="SIGNAL" class="0">
-<segment>
-<label x="78.74" y="109.22" size="1.778" layer="95" xref="yes"/>
-<wire x1="78.74" y1="109.22" x2="71.12" y2="109.22" width="0.1524" layer="91"/>
-<pinref part="U$2" gate="G$1" pin="D4"/>
-</segment>
 <segment>
 <pinref part="IC2" gate="A" pin="O"/>
 <wire x1="215.9" y1="144.78" x2="236.22" y2="144.78" width="0.1524" layer="91"/>
 <label x="236.22" y="144.78" size="1.778" layer="95" xref="yes"/>
+</segment>
+<segment>
+<label x="116.84" y="93.98" size="1.778" layer="95" xref="yes"/>
+<pinref part="U$2" gate="G$1" pin="D8"/>
+<wire x1="71.12" y1="93.98" x2="116.84" y2="93.98" width="0.1524" layer="91"/>
 </segment>
 </net>
@@
 <net name="WS2812_DATA" class="0">
 <segment>
-<label x="73.66" y="93.98" size="1.778" layer="95" xref="yes"/>
-<pinref part="U$2" gate="G$1" pin="D8"/>
-<wire x1="71.12" y1="93.98" x2="73.66" y2="93.98" width="0.1524" layer="91"/>
-</segment>
-<segment>
 <pinref part="LED" gate="G$1" pin="DIN"/>
 <wire x1="63.5" y1="154.94" x2="68.58" y2="154.94" width="0.1524" layer="91"/>
 <label x="68.58" y="154.94" size="1.778" layer="95" xref="yes"/>
 </segment>
+<segment>
+<label x="106.68" y="109.22" size="1.778" layer="95" xref="yes"/>
+<wire x1="106.68" y1="109.22" x2="71.12" y2="109.22" width="0.1524" layer="91"/>
+<pinref part="U$2" gate="G$1" pin="D4"/>
+</segment>
 </net>
